File: ads1298schield.brd (EAGLE design)
At the start: 101.6 x 53.3 mm, 85 parts, among them IC1 ADS1299IPAG, IC7 OPA376DBV, X1 SDBMF

Commit message: v0.4
Parts:
- removed D2: WHITE, SparkFun-LED:LED-1206
- removed IC7: OPA376DBV, OPA376:SOT23-5
- removed JP6: SRB1-BIAS, adafruit:1X03
- removed R22, R23: 2M, SparkFun-Passives:0603-RES
- removed R24: 4.99k, SparkFun-Passives:0603-RES
- removed U$4: (no value), SparkFun-Aesthetics:OSHW-LOGO-L
- removed U$7: (no value), endless-knot:ENDLESSKNOT-MEDIUM
- added C15: 10uF, SparkFun-Passives:1210
- added C16: 1.5nF, SparkFun-Passives:1210
- added C2: 100nF, rcl:C0603
- added C24: 22uF, SparkFun-Passives:1210
- added C26, C58, C59, C64: 100nF, rcl:C1210
- added C27: 1uF, SparkFun:0402-CAP
- added C3, C4: 4.7uF, SparkFun:0402-CAP
- added C5: 4.7uF, SteveMarple:EIA3216
- added C6: 10uF, SteveMarple:EIA3216
- added D4: red, SparkFun:LED-0603
- added JP1: LiPo, SparkFun:JST-2-SMD
- added JP58: SWD header, pinhead:1X04
- added L1, L2: 4.7uH, SteveMarple:1210-HAND
- added Q1: FDD4141TO252, transistor-fet:TO252
- added R11: 470, SparkFun:0402-RES
- added R12: 2k, SparkFun:0402-RES
- added R13: 976k, SteveMarple:1206-HAND
- added R14: 309k, SteveMarple:1206-HAND
- added R15: 340k, SteveMarple:1206-HAND
- added R16: 200k, SteveMarple:1206-HAND
- added R17: 15k, SteveMarple:1206-HAND
- added R27: 10k, resistor:M1406
- added R28: 100k, resistor:M1406
- added SW3: !RST, stm32f4stamp:SWITCH-TACT-B3U-1100P-B
- added U$2: ADS1298*PAG*, ADS129x:TQFP64
- added U1: MCP73831, SparkFun:SOT23-5
- added U2: LTC3440EMSPBF, LTC:SOP50P490X110-10N
- added X2: USB-MICROB, SparkFun:USB-MICROB
- C1: value (none) -> 1uF
- C60: value 1uF -> 100nF; device SparkFun-Passives:0603-CAP -> rcl:C1210
- C61: value 1uF -> 4.7uF; device SparkFun-Passives:0603-CAP -> rcl:C1210
- D1: value RED -> BAT60J; device SparkFun-LED:LED-1206 -> diode:SOD323_ST
- IC1: value ADS1299IPAG -> MCP1640SOT23-6-HAND; device ADS129x:TQFP64 -> SteveMarple:SOT23-6-HAND
- R1: value 270 -> 309k; device SparkFun-Passives:0603-RES -> SteveMarple:1206-HAND
- R10, R2, R3, R4, R5, R7, R8, R9: value (none) -> 10k
- R18: value 270 -> 2k; device SparkFun-Passives:0603-RES -> SparkFun:0402-RES
- U$1: value (none) -> BLUETOOTH-RN41"; device SparkFun-Aesthetics:OSHW-LOGO-L -> SparkFun:RN41
- U$3: value (none) -> STM32F411RE; device creative-commons:CC-BY-SA -> micro-stm_v3:LQFP64
- moved X1 211.2 mm to (133.3, 82.5), turned to 270 degrees
- moved R9 210.0 mm to (-54.6, 78.7)
- moved C1 205.5 mm to (-38.1, 85.1)
- moved R8 205.1 mm to (-48.3, 78.7)
- moved R10 204.9 mm to (-61.0, 78.7)
- moved R7 200.8 mm to (-41.9, 78.7)
- moved R5 197.3 mm to (-35.6, 78.7)
- moved R4 194.4 mm to (-29.2, 78.7)
- moved R3 192.4 mm to (-22.9, 78.7)
- moved U$10 174.3 mm to (-27.9, 100.3)
- moved U$9 172.9 mm to (-25.4, 100.3)
- moved U$8 171.6 mm to (-22.9, 100.3)
- moved R2 155.9 mm to (-16.5, 78.7)
- moved JP16 148.1 mm to (156.2, 16.5)
- moved C17 140.4 mm to (-76.2, 97.8), turned to 0 degrees
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Connections:
- removed net !PWDN: IC1.35
- removed net !RESET: IC1.36
- removed net !SPI_CS: IC1.39
- removed net AVDD: C10.1, C11.1, C12.1, C60.1, C7.1, C8.1, C9.1, IC1.19, IC1.21, IC1.22, IC1.54, IC1.56, IC1.59, IC7.5, JP16.2, R23.1
- removed net AVSS: C11.2, C12.2, C17.2, C18.2, C19.2, C20.2, C21.2, C29.2, C30.2, C61.2, C7.2, C8.2, IC1.20, IC1.23, IC1.32, IC1.53, IC1.57, IC1.58, IC7.2, R22.2
- removed net BIAS_ELEC: IC1.62, JP6.1, R24.2
- removed net BIAS_ELEC_CON: JP16.24, R24.1
- removed net BOARD_ADDR_0: IC1.42
- removed net BOARD_ADDR_1: IC1.44
- removed net BOARD_ADDR_2: IC1.45
- removed net CLK: IC1.37
- removed net CLKSEL: IC1.52
- removed net DRDY: IC1.47
- removed net DVDD: C13.1, C14.1, C25.1, C63.1, IC1.48, IC1.50, JP16.1, R1.1
- removed net GPIO4: IC1.46, R18.1
- removed net N$14: D2.A, R18.2
- removed net N$15: IC7.3, R22.1, R23.2
- removed net N$18: IC7.1, IC7.4, JP6.3
- removed net N$22: C66.2, R6.1
- removed net N$25: C66.1, IC1.63
- removed net N$7: R10.1
- removed net SPI_CLK: IC1.40
- removed net SPI_IN: IC1.34
- removed net SPI_OUT: IC1.43
- removed net SRB1: IC1.18, JP6.2
- removed net SRB2: IC1.17
- removed net START: IC1.38
- new net !DRDY1298: U$2.47, U$3.38
- new net !PWDN1298: U$2.35, U$3.57
- new net !RESET1298: U$2.36, U$3.58
- new net !SPI_CS1298: U$2.39, U$3.20
- new net +5V: C10.1, C11.1, C12.1, C6.A, C7.1, C8.1, C9.1, IC1.5, R13.2, U$2.19, U$2.21, U$2.22, U$2.54, U$2.56, U$2.59, U$2.60
- new net 5VIN: C3.1, D1.A, D4.A, Q1.1, R18.1, U1.4, X2.VBUS
- new net CLKSEL1298: U$2.52, U$3.59
- new net LINK: U$1.15, U$1.16
- new net N$100: R28.1, SW3.1, U$3.7
- new net N$13: C19.1, C20.1, U$2.55
- new net N$16: R12.1, U1.5
- new net N$17: R11.1, U1.1
- new net N$20: D4.C, R11.2
- new net N$21: IC1.1, L1.2
- new net N$23: C5.A, IC1.3, IC1.6, L1.1
- new net N$24: C16.1, U2.10
- new net N$26: IC1.4, R13.1, R14.2
- new net N$27: C15.1, U2.2, U2.7, U2.8
- new net N$28: L2.1, U2.3
- new net N$29: L2.2, U2.4
- new net N$31: R15.1, R16.2, R17.1, U2.9
- new net N$32: C16.2, R17.2
- new net N$87: C61.1, U$3.30
- new net N$98: R27.2, U$3.60
- new net N$99: C64.1, U$3.13
- new net RESET42: U$1.5, U$3.41
- new net RX-TX42: U$1.14, U$3.43
- new net SPI_CLK1298: U$2.40, U$3.21
- new net SPI_MISO1298: U$2.43, U$3.22
- new net SPI_MOSI1298: U$2.34, U$3.23
- new net START1298: U$2.38, U$3.37
- new net SWCLK: JP58.3, U$3.49
- new net SWDIO: JP58.4, U$3.46
- new net TX-RX42: U$1.13, U$3.42
- new net VBAT: C27.1, D1.C, Q1.2
- new net VBATT: C4.1, JP1.1, Q1.3, U1.3
- net +3V3: now also C13.1, C14.1, C2.1, C24.1, C25.1, C26.1, C58.1, C59.1, C60.1, C63.1, JP58.1, R10.1, R15.2, R28.2, U$1.11, U$2.48, U$2.50, U$3.1, U$3.19, U$3.32, U$3.48, U$3.64, U2.6
- net AGND: now also C11.2, C12.2, C15.2, C17.2, C18.2, C19.2, C2.2, C20.2, C21.2, C24.2, C26.2, C27.2, C29.2, C3.2, C30.2, C4.2, C5.C, C58.2, C59.2, C6.C, C61.2, C64.2, C7.2, C8.2, IC1.2, JP1.2, JP58.2, R1.1, R12.2, R14.1, R16.1, R18.2, R27.1, SW3.2, U$1.1, U$1.12, U$1.28, U$1.29, U$1.4, U$2.20, U$2.23, U$2.25, U$2.31, U$2.32, U$2.33, U$2.41, U$2.49, U$2.51, U$2.53, U$2.57, U$2.58, U$3.12, U$3.18, U$3.28, U$3.31, U$3.47, U$3.63, U1.2, U2.5, X2.GND; no longer C61.1, D1.C, D2.C, IC1.25, IC1.33, IC1.41, IC1.49, IC1.51, JP16.4, JP16.6
- net AIN1N: now also U$2.15; no longer IC1.15
- net AIN1P: now also U$2.16; no longer IC1.16
- net AIN2N: now also U$2.13; no longer IC1.13
- net AIN2P: now also U$2.14; no longer IC1.14
- net AIN3N: now also U$2.11; no longer IC1.11
- net AIN3P: now also U$2.12; no longer IC1.12
- net AIN4N: now also U$2.9; no longer IC1.9
- net AIN4P: now also U$2.10; no longer IC1.10
- net AIN5N: now also U$2.7; no longer IC1.7
- net AIN5P: now also U$2.8; no longer IC1.8
- net AIN6N: now also U$2.5; no longer IC1.5
- net AIN6P: now also U$2.6; no longer IC1.6
- net AIN7N: now also U$2.3; no longer IC1.3
- net AIN7P: now also U$2.4; no longer IC1.4
- net AIN8N: now also U$2.1; no longer IC1.1
- net AIN8P: now also U$2.2; no longer IC1.2
- net BIASINV: now also C66.2, R6.1, U$2.61; no longer IC1.61, R6.2
- net N$19: now also U2.1; no longer D1.A
- net N$3: now also U$2.28; no longer IC1.28
- net N$4: now also U$2.30; no longer IC1.30
- net N$5: now also C66.1, R6.2, U$2.62, U$2.63; no longer C19.1, C20.1, IC1.55
- net N$8: now also U$2.26; no longer IC1.26
- net VREFP: now also U$2.24; no longer IC1.24
Routing:
- net AVSS: track 164.5 -> 0.00 mm, vias 11 -> 0
- net AVDD: track 111.7 -> 0.00 mm, vias 5 -> 0
- net BIASINV: track 83.2 -> 0.00 mm, vias 2 -> 0
- net AGND: track 58.0 -> 0.00 mm, vias 28 -> 0
- net BOARD_ADDR_0: track 46.9 -> 0.00 mm, vias 4 -> 0
- net SRB1: track 46.0 -> 0.00 mm, vias 1 -> 0
- net BIAS_ELEC_CON: track 40.9 -> 0.00 mm, vias 1 -> 0
- net BOARD_ADDR_1: track 40.0 -> 0.00 mm, vias 2 -> 0
- net GPIO4: track 36.1 -> 0.00 mm, vias 2 -> 0
- net BOARD_ADDR_2: track 30.6 -> 0.00 mm, vias 2 -> 0
- net BIAS_ELEC: track 30.3 -> 0.00 mm, vias 1 -> 0
- net SRB2: track 28.2 -> 0.00 mm, vias 1 -> 0
- net AIN8N: track 20.6 -> 0.00 mm
- net AIN1P: track 20.0 -> 0.00 mm
- net AIN8P: track 19.4 -> 0.00 mm
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- removed copper zone on layer 2, net AGND
- removed copper zone on layer 1, net AVDD
- removed copper zone on layer 1, net AVSS
- removed copper zone on layer 16, net AVSS
- removed copper zone on layer 1, net BOARD_ADDR_0
- removed copper zone on layer 15, net DVDD
- removed copper zone on layer 1, net IOREF
- removed copper zone on layer 2, net N$12
- removed copper zone on layer 15, net N$23
- removed copper zone on layer 15, net N$26
- removed copper zone on layer 2, net N$55
- removed copper zone on layer 1, net REF_ELEC
- removed copper zone on layer 1, net SRB1
- removed copper zone on layer 1, net VCC_5V_FILTERED
Other:
- board size 101.6 x 53.3 mm -> 160 x 100 mm
- board text removed: "0"
- board text removed: "1"
- board text removed: "10"
- board text removed: "11"
- board text removed: "12"
- board text removed: "13"
- board text removed: "14"
- board text removed: "15"
- board text removed: "16"
- board text removed: "17"
- board text removed: "18"
- board text removed: "19"
- board text removed: "2"
- board text removed: "20"
- board text removed: "21"
- board text removed: "22"
- board text removed: "23"
- board text removed: "24"
- board text removed: "25"
- board text removed: "26"
- board text removed: "27"
- board text removed: "28"
- board text removed: "29"
- board text removed: "3"
- board text removed: "30"
- board text removed: "31"
- board text removed: "32"
- board text removed: "33"
- board text removed: "34"
- board text removed: "35"
- board text removed: "36"
- board text removed: "37"
- board text removed: "38"
- board text removed: "39"
- board text removed: "3V3"
- board text removed: "4"
- board text removed: "40"
- board text removed: "41"
- board text removed: "42"
- board text removed: "43"
- board text removed: "44"
- board text removed: "45"
- board text removed: "46"
- board text removed: "47"
- board text removed: "48"
- board text removed: "49"
- board text removed: "5"
- board text removed: "50"
- board text removed: "51"
- board text removed: "52"
- board text removed: "53"
- board text removed: "5V"
- board text removed: "6"
- board text removed: "7"
- board text removed: "8"
- board text removed: "9"
- board text removed: "A"
- board text removed: "A0"
- board text removed: "A1"
- board text removed: "A10"
- board text removed: "A11"
- board text removed: "A2"
- board text removed: "A3"
- board text removed: "A4"
- board text removed: "A5"
- board text removed: "A6"
- board text removed: "A7"
- board text removed: "A8"
- board text removed: "A9"
- board text removed: "AGND"
- board text removed: "AREF"
- board text removed: "AVDD"
- board text removed: "AVSS"
- board text removed: "B"
- board text removed: "BIASINV"
- board text removed: "Board Addr"
- board text removed: "CAN RX"
- board text removed: "CAN TX"
- board text removed: "CLK"
- board text removed: "DAC 0"
- board text removed: "DAC 1"
- board text removed: "DRDY"
- board text removed: "Electrodes"
- board text removed: "Ext. Sync"
- board text removed: "GND"
- board text removed: "GPIO4"
- board text removed: "HackEEG Shield"
- board text removed: "IOREF"
- board text removed: "Jumper Storage"
- board text removed: "Layer 1 Top signal"
- board text removed: "Layer 2 GND (-)"
- board text removed: "Layer 3 DVDD (+)"
- board text removed: "Layer 4 Bottom signal"
- board text removed: "MISO"
- board text removed: "MOSI"
- board text removed: "PWDN"
- board text removed: "Power"
- board text removed: "RESET"
- board text removed: "RST"
- board text removed: "Released under a Creative Commons Attribution-ShareAlike 4.0 Unported (CC BY-SA 4.0) license"
- board text removed: "SCK"
- board text removed: "SCL1"
- board text removed: "SCLK"
- board text removed: "SDA1"
- board text removed: "SPI CLK"
- board text removed: "SPI CS"
- board text removed: "SPI MISO"
- board text removed: "SPI MOSI"
- board text removed: "START"
- board text removed: "VIN"
- board text removed: "c 2014 Adam Feuer StarCat LLC"
- board text removed: "v1.3.1"

Commit message: v0.4
Parts:
- removed U$10, U$8, U$9: FIDUCIAL, adafruit:FIDUCIAL_1MM
- added C28, C32: 10uF, SparkFun-Passives:0603-CAP
- added C31: 220pF, SparkFun-Passives:0603-CAP
- added C33, C50: 4.7pF, SparkFun-Passives:0603-CAP
- added C51, C52, C53: 1uF, SparkFun-Passives:0603-CAP
- added D2: 0, diode:MELF-MLL41
- added IC2: ADS1258, mfePCB:P-HVQFN48-7X7
- added J1: 22-23-2091, con-molex:22-23-2091
- added L3: 6.8uH, SteveMarple:1210-HAND
- added R19: 1M, SparkFun-Passives:0603-RES
- added R20: 86.6k, SparkFun-Passives:0603-RES
- added R21: 10.2k, SparkFun-Passives:0603-RES
- added U$4: LMR62421, mfePCB:SOT23-5
- added X3: CRYSTALS-NOGND-91SMX, IQD-Frequency-Products:91SMX
- moved JP16 217.9 mm to (-57.1, 61.0), turned to 0 degrees
- moved U$1 216.3 mm to (-64.8, 7.62)
- moved X1 173.8 mm to (-27.9, 17.8), turned to 0 degrees
- moved D1 125.0 mm to (-19.1, 96.5)
- moved R18 120.5 mm to (-80.0, 109.2)
- moved C27 118.9 mm to (-68.6, 109.2)
- moved U$2 95.3 mm to (-20.3, 50.8)
- moved U$3 74.0 mm to (-38.1, 50.8), turned to 0 degrees
- moved C43 72.8 mm to (-87.6, 101.6)
- moved C44 72.8 mm to (-91.4, 101.6)
- moved R2 72.5 mm to (-88.9, 82.5)
- moved JP58 71.2 mm to (-38.1, 82.5), turned to 0 degrees
- moved C58 68.6 mm to (-85.1, 73.7)
- moved C59 68.6 mm to (-91.4, 73.7)
- moved R15 67.5 mm to (-82.5, 90.2)
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Connections:
- removed net VBATT: C4.1, JP1.1, Q1.3, U1.3
- new net !DRDY1258: IC2.25, U$3.34
- new net !PWDN1258: IC2.10, U$3.24
- new net !RESET1258: IC2.11, U$3.36
- new net !SPI_CS1258: IC2.27, U$3.33
- new net +12V: C28.1, C31.1, D2.C, J1.1, J1.2, J1.3, R20.2
- new net 4630ACCX: IC2.4, J1.4
- new net 4630ACCY: IC2.3, J1.5
- new net 4630ACCZ: IC2.2, J1.6
- new net CLKSEL1258: IC2.12, U$3.39
- new net N$12: C33.1, IC2.8, X3.2
- new net N$14: D2.A, L3.1, U$4.1
- new net N$15: C50.1, IC2.9, X3.1
- new net N$18: C31.2, R20.1, R21.2, U$4.3
- new net N$30: C53.1, IC2.31
- new net N$7: R19.1, U$4.4
- new net SPI_CLK1258: IC2.22, U$3.29
- new net SPI_MISO1258: IC2.24, U$3.10
- new net SPI_MOSI1258: IC2.23, U$3.11
- new net START1258: IC2.26, U$3.35
- net +3V3: now also C52.1, IC2.28
- net +5V: now also C51.1, IC2.6
- net AGND: now also C28.2, C32.2, C33.2, C50.2, C51.2, C52.2, C53.2, IC2.29, IC2.30, IC2.32, IC2.5, J1.7, J1.8, J1.9, R21.1, U$4.2
- net VBAT: now also C32.1, C4.1, JP1.1, L3.2, Q1.3, R19.2, U$4.5, U1.3
