File: ads1298schield.sch (EAGLE design)
At the start: 83 parts, among them IC7 OPA376DBV, X1 SDBMF

Commit message: v0.3
Parts:
- removed C61: 1uF, SparkFun-Passives:CAP0603-CAP
- removed D1: RED, SparkFun-LED:LED-RED1206
- removed R22, R23: 2M, SparkFun-Passives:RESISTOR0603-RES
- added C15: 10uF, SparkFun-Passives:CAP1210
- added C16: 1.5nF, SparkFun-Passives:CAP1210
- added C24: 22uF, SparkFun-Passives:CAP1210
- added C3, C4: 4.7uF, SparkFun:CAP0402-CAP
- added C5: 4.7uF, SteveMarple:CAP_POL1206
- added C6: 10uF, SteveMarple:CAP_POL1206
- added D4: red, SparkFun:LED0603
- added IC1: MCP1640SOT23-6-HAND, SteveMarple:MCP1640SOT23-6-HAND
- added JP1: LiPo, SparkFun:M02-JST-2MM-SMT
- added L1, L2: 4.7uH, SteveMarple:INDUCTOR1210-HAND
- added R11: 470, SparkFun:RESISTOR0402-RES
- added R12: 2k, SparkFun:RESISTOR0402-RES
- added R13: 976k, SteveMarple:RESISTOR1206-HAND
- added R14: 309k, SteveMarple:RESISTOR1206-HAND
- added R15: 340k, SteveMarple:RESISTOR1206-HAND
- added R16: 200k, SteveMarple:RESISTOR1206-HAND
- added R17: 15k, SteveMarple:RESISTOR1206-HAND
- added U1: MCP73831, SparkFun:MCP73831
- added U2: LTC3440EMSPBF, LTC:LTC3440EMSPBF
- added X2: USB-MICROB, SparkFun:USB-MICROB
- R1: value 270 -> 309k; device SparkFun-Passives:RESISTOR0603-RES -> SteveMarple:RESISTOR1206-HAND
Connections:
- removed net +3,3V: C2.1, U$1.VDD
- removed net 3.3V: U$2.AVDD1, U$2.AVDD_1, U$2.AVDD_2, U$2.AVDD_3, U$2.AVDD_4, U$2.AVDD_5
- removed net N$12 (its old number): U$1.GND, U$1.GND1, U$1.GND4, U$1.GND5, U$1.PIO7
- removed net N$15: IC7.P_IN, R22.1, R23.2
- new net +5V: C10.1, C11.1, C12.1, C6.+, C60.1, C7.1, C8.1, C9.1, IC1.VOUT, IC7.V_P, R13.2, U$2.AVDD1, U$2.AVDD_1, U$2.AVDD_2, U$2.AVDD_3, U$2.AVDD_4, U$2.AVDD_5
- new net 5VIN: C3.1, D4.A, U1.VIN, X2.VBUS
- new net N$16: R12.1, U1.PROG
- new net N$17: R11.1, U1.STAT
- new net N$20: D4.C, R11.2
- new net N$21: IC1.SW, L1.2
- new net N$23: C5.+, IC1.EN, IC1.VIN, L1.1
- new net N$24: C16.1, U2.VC
- new net N$26: IC1.VFB, R13.1, R14.2
- new net N$27: C15.1, U2.VIN, U2.~SHDN/SS
- new net N$28: L2.1, U2.SW1
- new net N$29: L2.2, U2.SW2
- new net N$31: R15.1, R16.2, R17.1, U2.FB
- new net N$32: C16.2, R17.2
- new net VBATT: C4.1, JP1.2, U1.VBAT
- net +3V3: now also C13.1, C14.1, C2.1, C24.1, C25.1, C63.1, R15.2, U$1.VDD, U2.VOUT
- net AGND: now also C11.2, C12.2, C15.2, C17.2, C18.2, C19.2, C20.2, C24.2, C29.2, C3.2, C30.2, C4.2, C5.-, C6.-, C7.2, C8.2, IC1.GND, IC7.V_N, JP1.1, R1.1, R12.2, R14.1, R16.1, U$1.GND, U$1.GND1, U$1.GND4, U$1.GND5, U$1.PIO7, U$2.AVSS1, U$2.AVSS_1, U$2.AVSS_2, U$2.AVSS_3, U$2.AVSS_4, U$2.AVSS_5, U1.VSS, U2.GND, X2.GND; no longer C29.1, C61.1, D1.C
- net AVDD: no longer C10.1, C11.1, C12.1, C60.1, C7.1, C8.1, C9.1, IC7.V_P, R23.1
- net AVSS: no longer C11.2, C12.2, C17.2, C18.2, C29.2, C30.2, C61.2, C7.2, C8.2, IC7.V_N, R22.2, U$2.AVSS1, U$2.AVSS_1, U$2.AVSS_2, U$2.AVSS_3, U$2.AVSS_4, U$2.AVSS_5
- net DVDD: no longer C13.1, C14.1, C25.1, C63.1, R1.1
- net GND: no longer C19.2, C20.2
- net N$19: now also U2.RT; no longer D1.A
Other:
- note added: "(This side to ADS1298 inputs)"
- note added: "3.3V buck-boost converter"
- note added: "5V boost converter"
- note added: "LiPo charger"
- note removed: "(This side to ADS1299 inputs)"
- note removed: "Power LED"
- moved on the sheet: C10, C11, C12, C13, C14, C25, C60, C63, C7, C8, C9, IC7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

Commit message: v0.3
Parts:
- removed C60: 1uF, SparkFun-Passives:CAP0603-CAP
- removed IC7: OPA376DBV, OPA376:OPA376DBV
- removed JP6: SRB1-BIAS, adafruit:PINHD-1X3
Connections:
- removed net N$12: IC7.N_IN, IC7.OUT, JP6.3
- net +5V: no longer C60.1, IC7.V_P
- net AGND: no longer C60.2, IC7.V_N
- net BIAS_ELEC: no longer JP6.1
- net N$5: now also U$2.RLD_IN
- net SRB1: no longer JP6.2
Other:
- note removed: "Bias"
- note removed: "Pins not labeled are not connected (NC)"
Changed lines of the file:
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@@
 <part name="SUPPLY40" library="supply2" deviceset="AGND" device=""/>
 <part name="D2" library="SparkFun-LED" deviceset="LED-WHITE" device="" value="WHITE"/>
-<part name="C60" library="SparkFun-Passives" deviceset="CAP" device="0603-CAP" value="1uF"/>
-<part name="SUPPLY46" library="supply2" deviceset="AGND" device=""/>
-<part name="JP6" library="adafruit" deviceset="PINHD-1X3" device="" value="SRB1-BIAS"/>
 <part name="R24" library="SparkFun-Passives" deviceset="RESISTOR" device="0603-RES" value="4.99k"/>
 <part name="R25" library="SparkFun-Passives" deviceset="RESISTOR" device="0603-RES" value="4.99k"/>
@@
 <part name="R6" library="SparkFun-Passives" deviceset="RESISTOR" device="0603-RES" value="3.98K"/>
 <part name="JP16" library="headers" deviceset="PINHD-2X12" device="" value="Electrodes"/>
-<part name="IC7" library="OPA376" deviceset="OPA376" device="DBV"/>
 <part name="U$8" library="adafruit" deviceset="FIDUCIAL" device=""/>
 <part name="U$9" library="adafruit" deviceset="FIDUCIAL" device=""/>
@@
 <part name="+3V6" library="supply1" deviceset="+3V3" device=""/>
 <part name="+3V7" library="supply1" deviceset="+3V3" device=""/>
-<part name="P+6" library="supply1" deviceset="+5V" device=""/>
-<part name="SUPPLY14" library="supply2" deviceset="AGND" device=""/>
 </parts>
 <sheets>
@@
 </segment>
 </net>
-<net name="BIAS_ELEC" class="0">
-<segment>
-<wire x1="304.8" y1="144.78" x2="304.8" y2="137.16" width="0.1524" layer="91"/>
-<label x="304.8" y="137.16" size="1.778" layer="95" rot="R270" xref="yes"/>
-</segment>
-</net>
 <net name="CLK" class="0">
 <segment>
@@
 <segment>
 <wire x1="309.88" y1="144.78" x2="309.88" y2="124.46" width="0.1524" layer="91"/>
-<label x="307.34" y="121.92" size="1.778" layer="95"/>
+<label x="307.34" y="127" size="1.778" layer="95"/>
 <pinref part="R6" gate="G$1" pin="2"/>
 <wire x1="302.26" y1="124.46" x2="309.88" y2="124.46" width="0.1524" layer="91"/>
@@
 <wire x1="284.48" y1="132.08" x2="307.34" y2="132.08" width="0.1524" layer="91"/>
 <pinref part="U$2" gate="G$1" pin="RLD_OUT"/>
-<wire x1="307.34" y1="132.08" x2="307.34" y2="144.78" width="0.1524" layer="91"/>
+<wire x1="307.34" y1="132.08" x2="307.34" y2="142.24" width="0.1524" layer="91"/>
+<pinref part="U$2" gate="G$1" pin="RLD_IN"/>
+<wire x1="307.34" y1="142.24" x2="307.34" y2="144.78" width="0.1524" layer="91"/>
+<wire x1="302.26" y1="144.78" x2="302.26" y2="142.24" width="0.1524" layer="91"/>
+<wire x1="302.26" y1="142.24" x2="307.34" y2="142.24" width="0.1524" layer="91"/>
 </segment>
 </net>
@@
 <plain>
 <text x="34.036" y="121.666" size="2.54" layer="91">Electrode Connector</text>
-<text x="293.116" y="179.324" size="2.54" layer="91">Bias</text>
 <text x="65.532" y="264.668" size="2.54" layer="91">Input Filtering</text>
 <text x="160.274" y="254.762" size="2.54" layer="91">(This side to ADS1298 inputs)</text>
 <text x="22.352" y="254.508" size="2.54" layer="91">(This side to electrode connector)</text>
 <text x="174.498" y="33.274" size="2.54" layer="91">Fiducials (for pick and place machines)</text>
-<text x="287.02" y="175.26" size="1.778" layer="91">Pins not labeled are not connected (NC)</text>
 </plain>
 <instances>
@@
 <attribute name="VALUE" x="112.649" y="18.415" size="1.778" layer="96"/>
 </instance>
-<instance part="C60" gate="G$1" x="304.8" y="193.04" smashed="yes" rot="MR270">
-<attribute name="NAME" x="305.689" y="188.468" size="1.778" layer="95" rot="MR0"/>
-<attribute name="VALUE" x="307.467" y="195.58" size="1.778" layer="96" rot="MR0"/>
-</instance>
-<instance part="SUPPLY46" gate="G$1" x="312.42" y="193.04" smashed="yes" rot="MR270">
-<attribute name="VALUE" x="315.468" y="193.04" size="1.778" layer="96" rot="MR180"/>
-</instance>
-<instance part="JP6" gate="A" x="259.08" y="226.06" rot="MR0"/>
 <instance part="R24" gate="G$1" x="81.026" y="143.51" smashed="yes">
 <attribute name="NAME" x="79.502" y="145.2626" size="1.778" layer="95"/>
@@
 </instance>
 <instance part="JP16" gate="A" x="53.34" y="157.226"/>
-<instance part="IC7" gate="G$1" x="297.18" y="220.98" rot="MR0"/>
 <instance part="U$8" gate="G$1" x="208.28" y="45.72"/>
 <instance part="U$9" gate="G$1" x="218.44" y="45.72"/>
 <instance part="U$10" gate="G$1" x="198.12" y="45.72"/>
-<instance part="P+6" gate="1" x="337.82" y="187.96" rot="R180"/>
-<instance part="SUPPLY14" gate="G$1" x="294.64" y="246.38" smashed="yes" rot="MR180">
-<attribute name="VALUE" x="294.005" y="249.047" size="1.778" layer="96" rot="MR90"/>
-</instance>
 </instances>
 <busses>
@@
 </segment>
 <segment>
-<pinref part="SUPPLY46" gate="G$1" pin="AGND"/>
-<pinref part="C60" gate="G$1" pin="2"/>
-<wire x1="309.88" y1="193.04" x2="307.34" y2="193.04" width="0.1524" layer="91"/>
-</segment>
-<segment>
 <pinref part="SUPPLY47" gate="G$1" pin="AGND"/>
 <pinref part="C62" gate="G$1" pin="2"/>
@@
 <label x="62.23" y="169.164" size="1.778" layer="95"/>
 <pinref part="JP16" gate="A" pin="4"/>
-</segment>
-<segment>
-<pinref part="IC7" gate="G$1" pin="V_N"/>
-<wire x1="294.64" y1="243.84" x2="294.64" y2="236.22" width="0.1524" layer="91"/>
-<pinref part="SUPPLY14" gate="G$1" pin="AGND"/>
 </segment>
 </net>
@@
 </segment>
 </net>
-<net name="SRB1" class="0">
-<segment>
-<pinref part="JP6" gate="A" pin="2"/>
-<wire x1="261.62" y1="226.06" x2="248.92" y2="226.06" width="0.1524" layer="91"/>
-<label x="248.92" y="226.06" size="1.27" layer="95"/>
-</segment>
-</net>
 <net name="REF_ELEC_CON" class="0">
 <segment>
@@
 <label x="85.852" y="143.764" size="1.778" layer="95"/>
 </segment>
-<segment>
-<pinref part="JP6" gate="A" pin="1"/>
-<wire x1="261.62" y1="228.6" x2="266.7" y2="228.6" width="0.1524" layer="91"/>
-<wire x1="266.7" y1="228.6" x2="266.7" y2="251.46" width="0.1524" layer="91"/>
-<label x="266.7" y="251.46" size="1.778" layer="95"/>
-</segment>
 </net>
 <net name="BIAS_ELEC_CON" class="0">
@@
 </segment>
 </net>
-<net name="+5V" class="0">
-<segment>
-<pinref part="P+6" gate="1" pin="+5V"/>
-<wire x1="337.82" y1="190.5" x2="337.82" y2="200.66" width="0.1524" layer="91"/>
-<wire x1="294.64" y1="200.66" x2="337.82" y2="200.66" width="0.1524" layer="91"/>
-<pinref part="IC7" gate="G$1" pin="V_P"/>
-<wire x1="294.64" y1="205.74" x2="294.64" y2="200.66" width="0.1524" layer="91"/>
-<wire x1="294.64" y1="200.66" x2="294.64" y2="193.04" width="0.1524" layer="91"/>
-<pinref part="C60" gate="G$1" pin="1"/>
-<wire x1="294.64" y1="193.04" x2="299.72" y2="193.04" width="0.1524" layer="91"/>
-</segment>
-</net>
-<net name="N$12" class="0">
-<segment>
-<pinref part="IC7" gate="G$1" pin="N_IN"/>
-<wire x1="312.42" y1="228.6" x2="314.96" y2="228.6" width="0.1524" layer="91"/>
-<wire x1="314.96" y1="228.6" x2="314.96" y2="238.76" width="0.1524" layer="91"/>
-<wire x1="314.96" y1="238.76" x2="279.4" y2="238.76" width="0.1524" layer="91"/>
-<wire x1="279.4" y1="238.76" x2="279.4" y2="223.52" width="0.1524" layer="91"/>
-<pinref part="IC7" gate="G$1" pin="OUT"/>
-<wire x1="281.94" y1="223.52" x2="279.4" y2="223.52" width="0.1524" layer="91"/>
-<pinref part="JP6" gate="A" pin="3"/>
-<wire x1="279.4" y1="223.52" x2="261.62" y2="223.52" width="0.1524" layer="91"/>
-</segment>
-</net>

Commit message: v0.3
Connections:
- removed net N$22: C66.2, R6.1
- net BIASINV: now also C66.2; no longer R6.2
- net N$5: now also R6.2
Other:
- moved on the sheet: R6
Changed lines of the file:
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@@
 <attribute name="VALUE" x="275.336" y="119.253" size="1.778" layer="96"/>
 </instance>
-<instance part="R6" gate="G$1" x="297.18" y="124.46" smashed="yes">
-<attribute name="NAME" x="298.45" y="126.2126" size="1.778" layer="95" rot="R90"/>
-<attribute name="VALUE" x="293.37" y="121.158" size="1.778" layer="96"/>
+<instance part="R6" gate="G$1" x="294.64" y="127" smashed="yes" rot="R90">
+<attribute name="NAME" x="292.8874" y="128.27" size="1.778" layer="95" rot="R180"/>
+<attribute name="VALUE" x="297.942" y="123.19" size="1.778" layer="96" rot="R90"/>
 </instance>
 <instance part="+3V3" gate="G$1" x="378.46" y="228.6"/>
@@
 <net name="BIASINV" class="0">
 <segment>
-<wire x1="309.88" y1="144.78" x2="309.88" y2="124.46" width="0.1524" layer="91"/>
+<wire x1="309.88" y1="144.78" x2="309.88" y2="121.92" width="0.1524" layer="91"/>
 <label x="307.34" y="127" size="1.778" layer="95"/>
-<pinref part="R6" gate="G$1" pin="2"/>
-<wire x1="302.26" y1="124.46" x2="309.88" y2="124.46" width="0.1524" layer="91"/>
-</segment>
-</net>
-<net name="N$22" class="0">
-<segment>
-<pinref part="R6" gate="G$1" pin="1"/>
-<wire x1="292.1" y1="124.46" x2="284.48" y2="124.46" width="0.1524" layer="91"/>
 <pinref part="C66" gate="G$1" pin="2"/>
+<wire x1="284.48" y1="124.46" x2="284.48" y2="121.92" width="0.1524" layer="91"/>
+<wire x1="284.48" y1="121.92" x2="309.88" y2="121.92" width="0.1524" layer="91"/>
 </segment>
 </net>
@@
 <segment>
 <pinref part="C66" gate="G$1" pin="1"/>
-<wire x1="284.48" y1="132.08" x2="307.34" y2="132.08" width="0.1524" layer="91"/>
+<wire x1="284.48" y1="132.08" x2="294.64" y2="132.08" width="0.1524" layer="91"/>
 <pinref part="U$2" gate="G$1" pin="RLD_OUT"/>
+<wire x1="294.64" y1="132.08" x2="307.34" y2="132.08" width="0.1524" layer="91"/>
 <wire x1="307.34" y1="132.08" x2="307.34" y2="142.24" width="0.1524" layer="91"/>
 <pinref part="U$2" gate="G$1" pin="RLD_IN"/>
@@
 <wire x1="302.26" y1="144.78" x2="302.26" y2="142.24" width="0.1524" layer="91"/>
 <wire x1="302.26" y1="142.24" x2="307.34" y2="142.24" width="0.1524" layer="91"/>
-</segment>
-</net>
+<pinref part="R6" gate="G$1" pin="2"/>
+<junction x="294.64" y="132.08"/>
+</segment>
+</net>

Commit message: v0.4
Parts:
- added C26, C58, C59, C60, C64: 100nF, rcl:C-EUC1210
- added C61: 4.7uF, rcl:C-EUC1210
- added JP58: (no value), pinhead:PINHD-1X4
- added R27: 10k, resistor:R-EU_M1406
- added R28: 100k, resistor:R-EU_M1406
- added SW3: !RST, stm32f4stamp:SWITCH-B3U-1110-BOSS
- added U$3: STM32F411RE, micro-stm_v3:STM32F411RE
Connections:
- new net N$100: R28.1, SW3..1, U$3G$1.NRST
- new net N$87: C61.1, U$3G$1.VCAP1
- new net N$88: C26.2
- new net N$91: C58.2
- new net N$92: C26.1
- new net N$93: C58.1
- new net N$94: C59.1
- new net N$95: C60.1
- new net N$96: C59.2
- new net N$97: C60.2
- new net N$98: R27.2, U$3G$1.BOOT0
- new net N$99: C64.1, U$3G$1.VDDA
- new net SWCLK: U$3G$1.PA14
- new net SWDIO: U$3G$1.PA13
- net +3V3: now also JP58.1, R28.2, U$3G$2.VDD@1, U$3G$2.VDD@2, U$3G$2.VDD@3, U$3G$2.VDD@4
- net AGND: now also C61.2, C64.2, R27.1, SW3..2, U$3G$1.BOOT1/PB2, U$3G$1.VSSA, U$3G$2.VSS@1, U$3G$2.VSS@4
Other:
- note added: "SWD debugger header"

Commit message: v0.4
Connections:
- net +3V3: now also U$3G$1.VBAT
Changed lines of the file:
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@@
 <part name="+3V10" library="supply1" deviceset="+3V3" device=""/>
 <part name="SUPPLY38" library="supply2" deviceset="AGND" device=""/>
+<part name="+3V11" library="supply1" deviceset="+3V3" device=""/>
 </parts>
 <sheets>
@@
 <instance part="+3V10" gate="G$1" x="20.32" y="66.04"/>
 <instance part="SUPPLY38" gate="G$1" x="-7.62" y="43.18"/>
+<instance part="+3V11" gate="G$1" x="30.48" y="45.72"/>
 </instances>
 <busses>
@@
 <pinref part="+3V10" gate="G$1" pin="+3V3"/>
 </segment>
-</net>
+<segment>
+<pinref part="+3V11" gate="G$1" pin="+3V3"/>
+<pinref part="U$3" gate="G$1" pin="VBAT"/>
+<wire x1="30.48" y1="43.18" x2="38.1" y2="43.18" width="0.1524" layer="91"/>
+</segment>
+</net>

Commit message: v0.4
Connections:
- removed net AVSS: C21.2
- removed net GND: C2.2
- removed net N$7: R10.1
- removed net N$88: C26.2
- removed net N$91: C58.2
- removed net N$92: C26.1
- removed net N$93: C58.1
- removed net N$94: C59.1
- removed net N$95: C60.1
- removed net N$96: C59.2
- removed net N$97: C60.2
- new net !DRDY1298: U$2.!DRDY, U$3G$1.PC7
- new net !PWDN1298: U$2.!PWDN, U$3G$1.PB5
- new net !RESET1298: U$2.!RESET, U$3G$1.PB6
- new net !SPI_CS1298: U$2.!CS, U$3G$1.PA4
- new net BOARD_ADDR_0: U$2.GPIO1
- new net BOARD_ADDR_1: U$2.GPIO2
- new net BOARD_ADDR_2: U$2.GPIO3
- new net CLKSEL1298: U$2.CLKSEL, U$3G$1.PB7
- new net N$15: C26.2, C58.2, C59.2, C60.2, U$3G$2.VDD@1, U$3G$2.VDD@2, U$3G$2.VDD@3, U$3G$2.VDD@4
- new net N$89: JP58.3
- new net N$90: JP58.4
- new net SPI_CLK1298: U$2.SCLK, U$3G$1.PA5
- new net SPI_MISO1298: U$2.DOUT, U$3G$1.PA6
- new net SPI_MOSI1298: U$2.DIN, U$3G$1.PA7
- new net START1298: U$2.START, U$3G$1.PC6
- net +3V3: now also C26.1, C58.1, C59.1, C60.1, R10.1; no longer U$3G$2.VDD@1, U$3G$2.VDD@2, U$3G$2.VDD@3, U$3G$2.VDD@4
- net +5V: now also U$2.RLD_REF
- net AGND: now also C2.2, C21.2, C23.2, C29.1, JP58.2, U$2.DAISY_IN, U$2.RESV1, U$3G$2.VSS@2, U$3G$2.VSS@3
- net BIASINV: now also R6.1, U$2.RLD_INV
- net GPIO4: now also U$2.GPIO4
- net N$27: now also U2.MODE/SYNC
- net N$3: now also U$2.VCAP1
- net N$4: now also U$2.VCAP2
Other:
- moved on the sheet: C26, C58, C59, C60

Commit message: v0.4
Parts:
- removed D2: WHITE, SparkFun-LED:LED-WHITE
- removed R24: 4.99k, SparkFun-Passives:RESISTOR0603-RES
- added C27: 1uF, SparkFun:CAP0402-CAP
- added D1: BAT60J, diode:BAT60J
- added Q1: FDD4141TO252, transistor-fet:FDD4141TO252
- C1: value (none) -> 1uF
- C2: value (none) -> 100nF
- JP58: value (none) -> SWD header
- R10, R2, R3, R4, R5, R7, R8, R9: value (none) -> 10k
- R18: value 270 -> 2k; device SparkFun-Passives:RESISTOR0603-RES -> SparkFun:RESISTOR0402-RES
Connections:
- removed net AVDD: JP16.2
- removed net BIAS_ELEC: R24.2
- removed net BIAS_ELEC_CON: JP16.24, R24.1
- removed net BOARD_ADDR_0: U$2.GPIO1
- removed net BOARD_ADDR_1: U$2.GPIO2
- removed net BOARD_ADDR_2: U$2.GPIO3
- removed net DVDD: JP16.1
- removed net GPIO4: R18.1, U$2.GPIO4
- removed net N$14: D2.A, R18.2
- removed net N$15: C26.2, C58.2, C59.2, C60.2, U$3G$2.VDD@1, U$3G$2.VDD@2, U$3G$2.VDD@3, U$3G$2.VDD@4
- removed net N$89: JP58.3
- removed net N$90: JP58.4
- removed net RESET: U$1.RESET
- removed net RX: U$1.UARTRX
- removed net SRB1: U$2.PACE_OUT2
- removed net SRB2: U$2.PACE_OUT1
- removed net TX: U$1.UARTTX
- new net RESET42: U$1.RESET, U$3G$1.PA8
- new net RX-TX42: U$1.UARTTX, U$3G$1.PA10
- new net TX-RX42: U$1.UARTRX, U$3G$1.PA9
- new net VBAT: C27.1, D1.C, Q1.S
- net +3V3: now also U$3G$2.VDD@1, U$3G$2.VDD@2, U$3G$2.VDD@3, U$3G$2.VDD@4
- net 5VIN: now also D1.A, Q1.G, R18.1
- net AGND: now also C26.2, C27.2, C58.2, C59.2, C60.2, JP1.2, R18.2; no longer D2.C, JP1.1, JP16.4, JP16.6
- net SWCLK: now also JP58.3
- net SWDIO: now also JP58.4
- net VBATT: now also JP1.1, Q1.D; no longer JP1.2
Other:
- note removed: "GPIO4 LED"
- note removed: "SWD debugger header"
- moved on the sheet: C26, C58, C59, C60, JP1, JP58, R18

Commit message: v0.4
Parts:
- removed U$10, U$8, U$9: FIDUCIAL, adafruit:FIDUCIAL
- added C28, C32: 10uF, SparkFun-Passives:CAP0603-CAP
- added C31: 220pF, SparkFun-Passives:CAP0603-CAP
- added C33, C50: 4.7pF, SparkFun-Passives:CAP0603-CAP
- added C51, C52, C53: 1uF, SparkFun-Passives:CAP0603-CAP
- added D2: 0, diode:DIODE-MELF-MLL41
- added IC2: ADS1258, mfePCB:ADS1258
- added J1, J2, J3: 22-23-2091, con-molex:22-23-2091
- added L3: 6.8uH, SteveMarple:INDUCTOR1210-HAND
- added R19: 1M, SparkFun-Passives:RESISTOR0603-RES
- added R20: 86.6k, SparkFun-Passives:RESISTOR0603-RES
- added R21: 10.2k, SparkFun-Passives:RESISTOR0603-RES
- added U$4: LMR62421, mfePCB:LMR62421
- added X3: CRYSTALS-NOGND-91SMX, IQD-Frequency-Products:CRYSTALS-NOGND-91SMX
Connections:
- removed net VBATT: C4.1, JP1.1, Q1.D, U1.VBAT
- new net !DRDY1258: IC2.!DRDY, U$3G$1.PB13
- new net !PWDN1258: IC2.!PWDN, U$3G$1.PC4
- new net !RESET1258: IC2.!RESET, U$3G$1.PB15
- new net !SPI_CS1258: IC2.!CS, U$3G$1.PB12
- new net +12V: C28.1, C31.1, D2.C, J1-1.S, J1-2.S, J1-3.S, R20.2
- new net 4630ACCX: IC2.AIN0, J1-4.S
- new net 4630ACCY: IC2.AIN1, J1-5.S
- new net 4630ACCZ: IC2.AIN2, J1-6.S
- new net ACCX1: IC2.AIN3, J2-2.S
- new net ACCX2: IC2.AIN8, J3-2.S
- new net ACCY1: IC2.AIN4, J2-3.S
- new net ACCY2: IC2.AIN9, J3-3.S
- new net ACCZ1: J2-4.S
- new net ACCZ2: IC2.AIN10, J3-4.S
- new net CLKSEL1258: IC2.CLKSEL, U$3G$1.PC8
- new net N$12: C33.1, IC2.XTAL1, X3.2
- new net N$14: D2.A, L3.1, U$4.SW
- new net N$15: C50.1, IC2.XTAL2, X3.1
- new net N$18: C31.2, R20.1, R21.2, U$4.FB
- new net N$22: J2-1.S
- new net N$25: J3-1.S
- new net N$30: C53.1, IC2.VREFP
- new net N$7: R19.1, U$4.SHDN
- new net ROTX1: J2-8.S
- new net ROTX2: IC2.AIN11, IC2.AIN12, J3-8.S
- new net ROTY1: J2-7.S
- new net ROTY2: IC2.AIN13, J3-7.S
- new net ROTZ1: J2-6.S
- new net ROTZ2: IC2.AIN14, J3-6.S
- new net SPI_CLK1258: IC2.SCLK, U$3G$1.PB10
- new net SPI_MISO1258: IC2.DOUT, U$3G$1.PC2
- new net SPI_MOSI1258: IC2.DIN, U$3G$1.PC3
- new net START1258: IC2.START, U$3G$1.PB14
- net +3V3: now also C52.1, IC2.DVDD
- net +5V: now also C51.1, IC2.AVDD
- net AGND: now also C28.2, C32.2, C33.2, C50.2, C51.2, C52.2, C53.2, IC2.AINCOM, IC2.AVSS, IC2.DGND, IC2.VREFN, J1-7.S, J1-8.S, J1-9.S, J2-5.S, J3-5.S, R21.1, U$4.GND
- net VBAT: now also C32.1, C4.1, JP1.1, L3.2, Q1.D, R19.2, U$4.VIN, U1.VBAT
Other:
- note added: "4630A connector"
- note added: "6DOF module #1"
- note added: "6DOF module #2"
- note added: "Boost converter for 4630A accelerometer"
- note removed: "Fiducials (for pick and place machines)"
